File: H1DR10/Design/H1DR10.brd (EAGLE design)
At the start: 34.6 x 30 mm, 21 parts, among them P1 HEXABIT_17.32_NO_P6, U1 STM32F091CBU6, X1 XTALL_CSTCE8M00G52

Commit message: full unchecked
Parts:
- added C10, C12: 100nF, Hexabitz:C-0603
- added C11: 4.7uF, Hexabitz:C-0805-POL
- added P2: RS-485, Hexabitz:1546111-2
- added R4, R7: 0.0R, Hexabitz:R-0603
- added R5: 120R, Hexabitz:R-0805
- added R6: 10k, Hexabitz:R-0603
- added U2: MAX14840EASAT, Hexabitz:SOIC127P600X175-8N
- C1: value 10nF -> 100nF
- C3: value 100nF -> 4.7uF; device Hexabitz:C-0603 -> Hexabitz:C-0805-POL
- C5: value 100nF -> 10nF
- C7: value 4.7uF -> 100nF; device Hexabitz:C-0805-POL -> Hexabitz:C-0603
- D1: value VLMS1300-GS08 -> RED
- moved C5 14.1 mm to (41.8, 31.5)
- moved B 13.2 mm to (24.9, 44.5)
- moved C 12.8 mm to (22.8, 34.6)
- moved D 12.8 mm to (22.8, 32.1)
- moved R 11.8 mm to (48.2, 32.0)
- moved FB1 10.2 mm to (42.2, 25.2), turned to 270 degrees
- moved C3 10.1 mm to (27.6, 38.1), turned to 270 degrees
- moved C7 8.63 mm to (29.6, 31.5)
- moved C6 8.49 mm to (29.6, 38.2), turned to 270 degrees
- moved D1 7.14 mm to (28.3, 24.9), turned to 0 degrees
- moved R1 6.84 mm to (28.4, 27.9)
- moved C8 5.63 mm to (38.0, 39.9), turned to 0 degrees
- moved C1 4.67 mm to (44.1, 35.1)
- moved C9 1.64 mm to (39.6, 37.3), turned to 270 degrees
- moved X1 1.45 mm to (41.8, 35.1)
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Connections:
- new net N$10: R4.1, R5.2
- new net N$2: C12.2, R4.2, R7.1
- new net N$7: P2.2, R5.1, U2.7
- new net N$8: C12.1, P2.1, R7.2, U2.6
- new net UART1_RTS: R6.1, U1.P$33, U2.2, U2.3
- net GND: now also C1.2, C10.2, C11.2, R6.2, U1.P$2, U1.P$20, U2.5; no longer C5.2
- net R1: now also C1.1; no longer C8.1
- net UART1_RX: now also U2.4
- net UART1_TX: now also U2.1
- net UART2_RX: now also P1.PAD_PD2
- net UART2_TX: now also P1.PAD_PU2
- net UART3_RX: now also P1.PAD_PD4
- net UART3_TX: now also P1.PAD_PU4
- net UART4_RX: now also P1.PAD_PD1
- net UART4_TX: now also P1.PAD_PU1
- net UART5_RX: now also P1.PAD_PD5
- net UART5_TX: now also P1.PAD_PU5
- net UART6_RX: now also P1.PAD_PD3
- net UART6_TX: now also P1.PAD_PU3
- net VDD: now also C10.1, C11.1, C8.1, U2.8; no longer C5.1
- net VDDA: now also C5.1; no longer C1.1
- net VSSA: now also C5.2; no longer C1.2
Routing:
- net UART4_RX: track 0.00 -> 23.6 mm
- net UART4_TX: track 0.00 -> 23.0 mm, vias 0 -> 1
- net UART1_RTS: track 0.00 -> 21.8 mm, vias 0 -> 1
- net N$8: track 0.00 -> 20.6 mm
- net UART1_RX: track 0.00 -> 19.0 mm, vias 0 -> 1
- net VDD: track 0.00 -> 18.3 mm, vias 0 -> 3
- net GND: track 0.00 -> 18.1 mm, vias 0 -> 6
- net N$9: track 0.00 -> 16.7 mm, vias 0 -> 1
- net B1: track 0.00 -> 15.5 mm, vias 0 -> 1
- net R1: track 0.00 -> 14.6 mm, vias 0 -> 2
- net UART5_RX: track 0.00 -> 14.5 mm
- net UART3_TX: track 0.00 -> 13.8 mm, vias 0 -> 1
- net UART5_TX: track 0.00 -> 13.1 mm, vias 0 -> 1
- net UART6_TX: track 0.00 -> 12.8 mm, vias 0 -> 1
- net UART3_RX: track 0.00 -> 12.8 mm
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Other:
- board text added: "DC Term"
- board text added: "P2*"
- board text added: "TA"
- board text added: "TB"
- board text removed: "P2"
