File: H1DR10/Design/H1DR10.sch (EAGLE design)
At the start: 21 parts, among them P1 HEXABIT_17.32_NO_P6, U1 STM32F091CBU6, X1 XTALL_CSTCE8M00G52

Commit message: full unchecked
Parts:
- added C10, C12: 100nF, Hexabitz:C-0603
- added C11: 4.7uF, Hexabitz:C-0805-POL
- added P2: RS-485, Hexabitz:1546111-2
- added R4, R7: 0.0R, Hexabitz:R-0603
- added R5: 120R, Hexabitz:R-0805
- added R6: 10k, Hexabitz:R-0603
- added U2: MAX14840EASAT, Hexabitz:MAX14840EASAT
- C1: value 10nF -> 100nF; CAPACITANCE 10nF -> 100nF; MPN C0603C103K5RACTU -> C0603C104K8RACTU; OCTOPART_URL https://octopart.com/c0603c103k5ractu-kemet-133094?r=sp&s=R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 -> https://octopart.com/c0603c104k8ractu-kemet-145075?r=sp&s=9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; VOLTAGE_RATING 50V -> 10V
- C3: value 100nF -> 4.7uF; device Hexabitz:C-0603 -> Hexabitz:C-0805-POL; CAPACITANCE 100nF -> 4.7uF; MFN KEMET -> Murata; MPN C0603C104K8RACTU -> GRM21BC81E475KA12L; OCTOPART_URL https://octopart.com/c0603c104k8ractu-kemet-145075?r=sp&s=9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 -> https://octopart.com/grm21bc81e475ka12l-murata-10331911?r=s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; VOLTAGE_RATING 10V -> 25V
- C5: value 100nF -> 10nF; CAPACITANCE 100nF -> 10nF; MPN C0603C104K8RACTU -> C0603C103K5RACTU; OCTOPART_URL https://octopart.com/c0603c104k8ractu-kemet-145075?r=sp&s=9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 -> https://octopart.com/c0603c103k5ractu-kemet-133094?r=sp&s=R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; VOLTAGE_RATING 10 -> 50V
- C7: value 4.7uF -> 100nF; device Hexabitz:C-0805-POL -> Hexabitz:C-0603; CAPACITANCE 4.7uF -> 100nF; MFN Murata -> KEMET; MPN GRM21BC81E475KA12L -> C0603C104K8RACTU; OCTOPART_URL https://octopart.com/grm21bc81e475ka12l-murata-10331911?r=s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 -> https://octopart.com/c0603c104k8ractu-kemet-145075?r=sp&s=9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; VOLTAGE_RATING 25V -> 10
- D1: value VLMS1300-GS08 -> RED
Connections:
- new net N$10: R4.1, R5.2
- new net N$2: C12.2, R4.2, R7.1
- new net N$7: P2.2, R5.1, U2.B
- new net N$8: C12.1, P2.1, R7.2, U2.A
- new net UART1_RTS: R6.1, U1.PA12, U2.!RE, U2.DE
- net GND: now also C1.2, C10.2, C11.-, C3.-, C7.2, R6.2, U1.PB2, U1.PC13, U2.GND; no longer C3.2, C5.2, C7.-
- net R1: now also C1.1; no longer C8.1
- net UART1_RX: now also U2.DI
- net UART1_TX: now also U2.RO
- net UART2_RX: now also P1.SD2
- net UART2_TX: now also P1.SU2
- net UART3_RX: now also P1.SD4
- net UART3_TX: now also P1.SU4
- net UART4_RX: now also P1.SD1
- net UART4_TX: now also P1.SU1
- net UART5_RX: now also P1.SD5
- net UART5_TX: now also P1.SU5
- net UART6_RX: now also P1.SD3
- net UART6_TX: now also P1.SU3
- net VDD: now also C10.1, C11.+, C3.+, C7.1, C8.1, U2.VCC; no longer C3.1, C5.1, C7.+
- net VDDA: now also C5.1; no longer C1.1
- net VSSA: now also C5.2; no longer C1.2
Other:
- note added: "Amir Tabbakh"
- note added: "RS485 Serial Transceiver"
- note removed: "Add Description Here"
- moved on the sheet: C, C1, C4, C5, C6, C8, D, D1, R1, X1
