File: H1DR1x-T/Design/H1DR1x-T.sch (EAGLE design)
At the start: 30 parts, among them P1 HEXABIT_17.32_NO_P6, P2 RS-485, U1 STM32G0B1CEU6QFN_B1CEU6_STM-L, U2 MAX14840EASAT, X1 XTALL_CSTCE8M00G52

Commit message: - Drew PCB.
Parts:
- renumbered ORANGE to ORG, YELLOW to YLW
Connections:
- net USART3_RX: now also P1.SD5; no longer P1.SD4
- net USART3_TX: now also P1.SU5; no longer P1.SU4
- net USART4_RX: now also P1.SD3; no longer P1.SD1
- net USART4_TX: now also P1.SU3; no longer P1.SU1
- net USART5_RX: now also P1.SD4; no longer P1.SD5
- net USART5_TX: now also P1.SU4; no longer P1.SU5
- net USART6_RX: now also P1.SD1; no longer P1.SD3
- net USART6_TX: now also P1.SU1; no longer P1.SU3
Changed lines of the file:
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@@
 <part name="R8" library="HEXABITZ_RCLS" library_urn="urn:adsk.eagle:library:20064561" deviceset="R-0603" device="" package3d_urn="urn:adsk.eagle:package:1435818/6" value="270.0R"/>
 <part name="R9" library="HEXABITZ_RCLS" library_urn="urn:adsk.eagle:library:20064561" deviceset="R-0603" device="" package3d_urn="urn:adsk.eagle:package:1435818/6" value="270.0R"/>
-<part name="YELLOW" library="HEXABITZ_USER_INTERFACE_PARTS" library_urn="urn:adsk.eagle:library:20064563" deviceset="LED" device="CHIP-LED0805" package3d_urn="urn:adsk.eagle:package:15818/2"/>
-<part name="ORANGE" library="HEXABITZ_USER_INTERFACE_PARTS" library_urn="urn:adsk.eagle:library:20064563" deviceset="LED" device="CHIP-LED0805" package3d_urn="urn:adsk.eagle:package:15818/2"/>
+<part name="YLW" library="HEXABITZ_USER_INTERFACE_PARTS" library_urn="urn:adsk.eagle:library:20064563" deviceset="LED" device="CHIP-LED0805" package3d_urn="urn:adsk.eagle:package:15818/2"/>
+<part name="ORG" library="HEXABITZ_USER_INTERFACE_PARTS" library_urn="urn:adsk.eagle:library:20064563" deviceset="LED" device="CHIP-LED0805" package3d_urn="urn:adsk.eagle:package:15818/2"/>
 <part name="GND4" library="supply1" library_urn="urn:adsk.eagle:library:371" deviceset="GND" device=""/>
 <part name="GND7" library="supply1" library_urn="urn:adsk.eagle:library:371" deviceset="GND" device=""/>
@@
 <attribute name="VALUE" x="226.06" y="170.307" size="1.778" layer="96" rot="R180"/>
 </instance>
-<instance part="YELLOW" gate="G$1" x="236.22" y="175.26" smashed="yes" rot="R90">
+<instance part="YLW" gate="G$1" x="236.22" y="175.26" smashed="yes" rot="R90">
 <attribute name="NAME" x="240.792" y="178.816" size="1.778" layer="95" rot="R180"/>
 <attribute name="VALUE" x="240.792" y="180.975" size="1.778" layer="96" rot="R180"/>
 </instance>
-<instance part="ORANGE" gate="G$1" x="236.22" y="167.005" smashed="yes" rot="R90">
+<instance part="ORG" gate="G$1" x="236.22" y="167.005" smashed="yes" rot="R90">
 <attribute name="NAME" x="240.792" y="170.561" size="1.778" layer="95" rot="R180"/>
 <attribute name="VALUE" x="240.792" y="172.72" size="1.778" layer="96" rot="R180"/>
@@
 <segment>
 <pinref part="GND4" gate="1" pin="GND"/>
-<pinref part="ORANGE" gate="G$1" pin="C"/>
+<pinref part="ORG" gate="G$1" pin="C"/>
 <wire x1="244.475" y1="166.37" x2="244.475" y2="167.005" width="0.1524" layer="91"/>
 <wire x1="244.475" y1="167.005" x2="241.3" y2="167.005" width="0.1524" layer="91"/>
 </segment>
 <segment>
-<pinref part="YELLOW" gate="G$1" pin="C"/>
+<pinref part="YLW" gate="G$1" pin="C"/>
 <pinref part="GND7" gate="1" pin="GND"/>
 <wire x1="241.3" y1="175.26" x2="256.54" y2="175.26" width="0.1524" layer="91"/>
@@
 <net name="USART4_TX" class="0">
 <segment>
-<pinref part="P1" gate="G$1" pin="SU1"/>
-<wire x1="68.58" y1="172.72" x2="81.28" y2="172.72" width="0.1524" layer="91"/>
-<label x="68.58" y="172.72" size="1.778" layer="95"/>
-</segment>
-<segment>
 <pinref part="U1" gate="A" pin="PA0"/>
 <wire x1="140.335" y1="162.56" x2="123.825" y2="162.56" width="0.1524" layer="91"/>
 <label x="123.825" y="162.56" size="1.778" layer="95"/>
 </segment>
+<segment>
+<pinref part="P1" gate="G$1" pin="SU3"/>
+<wire x1="68.58" y1="162.56" x2="81.28" y2="162.56" width="0.1524" layer="91"/>
+<label x="68.58" y="162.56" size="1.778" layer="95"/>
+</segment>
 </net>
 <net name="USART4_RX" class="0">
-<segment>
-<pinref part="P1" gate="G$1" pin="SD1"/>
-<wire x1="68.58" y1="137.16" x2="81.28" y2="137.16" width="0.1524" layer="91"/>
-<label x="68.58" y="137.16" size="1.778" layer="95"/>
-</segment>
 <segment>
 <pinref part="U1" gate="A" pin="PA1"/>
@@
 <label x="123.825" y="160.02" size="1.778" layer="95"/>
 </segment>
+<segment>
+<pinref part="P1" gate="G$1" pin="SD3"/>
+<wire x1="68.58" y1="127" x2="81.28" y2="127" width="0.1524" layer="91"/>
+<label x="68.58" y="127" size="1.778" layer="95"/>
+</segment>
 </net>
 <net name="USART3_TX" class="0">
@@
 </segment>
 <segment>
-<pinref part="P1" gate="G$1" pin="SU4"/>
-<wire x1="68.58" y1="157.48" x2="81.28" y2="157.48" width="0.1524" layer="91"/>
-<label x="68.58" y="157.48" size="1.778" layer="95"/>
+<pinref part="P1" gate="G$1" pin="SU5"/>
+<wire x1="68.58" y1="152.4" x2="81.28" y2="152.4" width="0.1524" layer="91"/>
+<label x="68.58" y="152.4" size="1.778" layer="95"/>
 </segment>
 </net>
@@
 </segment>
 <segment>
-<pinref part="P1" gate="G$1" pin="SD4"/>
-<wire x1="68.58" y1="121.92" x2="81.28" y2="121.92" width="0.1524" layer="91"/>
-<label x="68.58" y="121.92" size="1.778" layer="95"/>
+<pinref part="P1" gate="G$1" pin="SD5"/>
+<wire x1="68.58" y1="116.84" x2="81.28" y2="116.84" width="0.1524" layer="91"/>
+<label x="68.58" y="116.84" size="1.778" layer="95"/>
 </segment>
 </net>
@@
 </segment>
 <segment>
-<pinref part="P1" gate="G$1" pin="SU3"/>
-<wire x1="68.58" y1="162.56" x2="81.28" y2="162.56" width="0.1524" layer="91"/>
-<label x="68.58" y="162.56" size="1.778" layer="95"/>
+<pinref part="P1" gate="G$1" pin="SU1"/>
+<wire x1="68.58" y1="172.72" x2="81.28" y2="172.72" width="0.1524" layer="91"/>
+<label x="68.58" y="172.72" size="1.778" layer="95"/>
 </segment>
 </net>
@@
 </segment>
 <segment>
-<pinref part="P1" gate="G$1" pin="SD3"/>
-<wire x1="68.58" y1="127" x2="81.28" y2="127" width="0.1524" layer="91"/>
-<label x="68.58" y="127" size="1.778" layer="95"/>
+<pinref part="P1" gate="G$1" pin="SD1"/>
+<wire x1="68.58" y1="137.16" x2="81.28" y2="137.16" width="0.1524" layer="91"/>
+<label x="68.58" y="137.16" size="1.778" layer="95"/>
 </segment>
 </net>
@@
 </segment>
 <segment>
-<pinref part="P1" gate="G$1" pin="SD5"/>
-<wire x1="68.58" y1="116.84" x2="81.28" y2="116.84" width="0.1524" layer="91"/>
-<label x="68.58" y="116.84" size="1.778" layer="95"/>
+<pinref part="P1" gate="G$1" pin="SD4"/>
+<wire x1="68.58" y1="121.92" x2="81.28" y2="121.92" width="0.1524" layer="91"/>
+<label x="68.58" y="121.92" size="1.778" layer="95"/>
 </segment>
 </net>
@@
 </segment>
 <segment>
-<pinref part="P1" gate="G$1" pin="SU5"/>
-<wire x1="68.58" y1="152.4" x2="81.28" y2="152.4" width="0.1524" layer="91"/>
-<label x="68.58" y="152.4" size="1.778" layer="95"/>
+<pinref part="P1" gate="G$1" pin="SU4"/>
+<wire x1="68.58" y1="157.48" x2="81.28" y2="157.48" width="0.1524" layer="91"/>
+<label x="68.58" y="157.48" size="1.778" layer="95"/>
 </segment>
 </net>
@@
 <segment>
 <pinref part="R9" gate="G$1" pin="1"/>
-<pinref part="ORANGE" gate="G$1" pin="A"/>
+<pinref part="ORG" gate="G$1" pin="A"/>
 <wire x1="228.6" y1="167.005" x2="233.68" y2="167.005" width="0.1524" layer="91"/>
 </segment>
@@
 <segment>
 <pinref part="R8" gate="G$1" pin="1"/>
-<pinref part="YELLOW" gate="G$1" pin="A"/>
+<pinref part="YLW" gate="G$1" pin="A"/>
 <wire x1="228.6" y1="175.26" x2="233.68" y2="175.26" width="0.1524" layer="91"/>
 </segment>

Commit message: - Regenerated Documentation. - BOM is ready. - Regenerated output files.
Parts:
- removed ORG: (no value), HEXABITZ_USER_INTERFACE_PARTS:LEDCHIP-LED0805
- added D3: Orange, HEXABITZ_USER_INTERFACE_PARTS:LEDCHIP-LED0805
- D2: value (none) -> Yellow
- renumbered YLW to D2
Connections:
- net GND: now also D3.C; no longer ORG.C
- net N$12: now also D3.A; no longer ORG.A
Other:
- moved on the sheet: R9
Changed lines of the file:
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@@
 <part name="R8" library="HEXABITZ_RCLS" library_urn="urn:adsk.eagle:library:20064561" deviceset="R-0603" device="" package3d_urn="urn:adsk.eagle:package:1435818/6" value="270.0R"/>
 <part name="R9" library="HEXABITZ_RCLS" library_urn="urn:adsk.eagle:library:20064561" deviceset="R-0603" device="" package3d_urn="urn:adsk.eagle:package:1435818/6" value="270.0R"/>
-<part name="YLW" library="HEXABITZ_USER_INTERFACE_PARTS" library_urn="urn:adsk.eagle:library:20064563" deviceset="LED" device="CHIP-LED0805" package3d_urn="urn:adsk.eagle:package:15818/2"/>
-<part name="ORG" library="HEXABITZ_USER_INTERFACE_PARTS" library_urn="urn:adsk.eagle:library:20064563" deviceset="LED" device="CHIP-LED0805" package3d_urn="urn:adsk.eagle:package:15818/2"/>
+<part name="D2" library="HEXABITZ_USER_INTERFACE_PARTS" library_urn="urn:adsk.eagle:library:20064563" deviceset="LED" device="CHIP-LED0805" package3d_urn="urn:adsk.eagle:package:15818/2" value="Yellow"/>
+<part name="D3" library="HEXABITZ_USER_INTERFACE_PARTS" library_urn="urn:adsk.eagle:library:20064563" deviceset="LED" device="CHIP-LED0805" package3d_urn="urn:adsk.eagle:package:15818/2" value="Orange"/>
 <part name="GND4" library="supply1" library_urn="urn:adsk.eagle:library:371" deviceset="GND" device=""/>
 <part name="GND7" library="supply1" library_urn="urn:adsk.eagle:library:371" deviceset="GND" device=""/>
@@
 <attribute name="VALUE" x="226.06" y="178.562" size="1.778" layer="96" rot="R180"/>
 </instance>
-<instance part="R9" gate="G$1" x="223.52" y="167.005" smashed="yes" rot="R180">
-<attribute name="NAME" x="225.425" y="165.5064" size="1.778" layer="95" rot="R180"/>
-<attribute name="VALUE" x="226.06" y="170.307" size="1.778" layer="96" rot="R180"/>
-</instance>
-<instance part="YLW" gate="G$1" x="236.22" y="175.26" smashed="yes" rot="R90">
+<instance part="R9" gate="G$1" x="223.52" y="165.735" smashed="yes" rot="R180">
+<attribute name="NAME" x="225.425" y="164.2364" size="1.778" layer="95" rot="R180"/>
+<attribute name="VALUE" x="226.06" y="169.037" size="1.778" layer="96" rot="R180"/>
+</instance>
+<instance part="D2" gate="G$1" x="236.22" y="175.26" smashed="yes" rot="R90">
 <attribute name="NAME" x="240.792" y="178.816" size="1.778" layer="95" rot="R180"/>
 <attribute name="VALUE" x="240.792" y="180.975" size="1.778" layer="96" rot="R180"/>
 </instance>
-<instance part="ORG" gate="G$1" x="236.22" y="167.005" smashed="yes" rot="R90">
-<attribute name="NAME" x="240.792" y="170.561" size="1.778" layer="95" rot="R180"/>
-<attribute name="VALUE" x="240.792" y="172.72" size="1.778" layer="96" rot="R180"/>
-</instance>
-<instance part="GND4" gate="1" x="244.475" y="163.83" smashed="yes" rot="MR0">
-<attribute name="VALUE" x="247.015" y="161.29" size="1.778" layer="96" rot="MR0"/>
-</instance>
-<instance part="GND7" gate="1" x="256.54" y="163.83" smashed="yes" rot="MR0">
-<attribute name="VALUE" x="259.08" y="161.29" size="1.778" layer="96" rot="MR0"/>
+<instance part="D3" gate="G$1" x="236.22" y="165.735" smashed="yes" rot="R90">
+<attribute name="NAME" x="240.792" y="169.291" size="1.778" layer="95" rot="R180"/>
+<attribute name="VALUE" x="240.792" y="171.45" size="1.778" layer="96" rot="R180"/>
+</instance>
+<instance part="GND4" gate="1" x="244.475" y="161.29" smashed="yes" rot="MR0">
+<attribute name="VALUE" x="247.015" y="158.75" size="1.778" layer="96" rot="MR0"/>
+</instance>
+<instance part="GND7" gate="1" x="256.54" y="161.29" smashed="yes" rot="MR0">
+<attribute name="VALUE" x="259.08" y="158.75" size="1.778" layer="96" rot="MR0"/>
 </instance>
 </instances>
@@
 <segment>
 <pinref part="GND4" gate="1" pin="GND"/>
-<pinref part="ORG" gate="G$1" pin="C"/>
-<wire x1="244.475" y1="166.37" x2="244.475" y2="167.005" width="0.1524" layer="91"/>
-<wire x1="244.475" y1="167.005" x2="241.3" y2="167.005" width="0.1524" layer="91"/>
-</segment>
-<segment>
-<pinref part="YLW" gate="G$1" pin="C"/>
+<pinref part="D3" gate="G$1" pin="C"/>
+<wire x1="244.475" y1="163.83" x2="244.475" y2="165.735" width="0.1524" layer="91"/>
+<wire x1="244.475" y1="165.735" x2="241.3" y2="165.735" width="0.1524" layer="91"/>
+</segment>
+<segment>
+<pinref part="D2" gate="G$1" pin="C"/>
 <pinref part="GND7" gate="1" pin="GND"/>
 <wire x1="241.3" y1="175.26" x2="256.54" y2="175.26" width="0.1524" layer="91"/>
-<wire x1="256.54" y1="175.26" x2="256.54" y2="166.37" width="0.1524" layer="91"/>
+<wire x1="256.54" y1="175.26" x2="256.54" y2="163.83" width="0.1524" layer="91"/>
 </segment>
 </net>
@@
 <pinref part="U1" gate="A" pin="PB4"/>
 <wire x1="211.455" y1="172.72" x2="215.265" y2="172.72" width="0.1524" layer="91"/>
-<wire x1="215.265" y1="172.72" x2="215.265" y2="167.005" width="0.1524" layer="91"/>
+<wire x1="215.265" y1="172.72" x2="215.265" y2="165.735" width="0.1524" layer="91"/>
 <pinref part="R9" gate="G$1" pin="2"/>
-<wire x1="215.265" y1="167.005" x2="218.44" y2="167.005" width="0.1524" layer="91"/>
+<wire x1="215.265" y1="165.735" x2="218.44" y2="165.735" width="0.1524" layer="91"/>
 </segment>
 </net>
@@
 <segment>
 <pinref part="R9" gate="G$1" pin="1"/>
-<pinref part="ORG" gate="G$1" pin="A"/>
-<wire x1="228.6" y1="167.005" x2="233.68" y2="167.005" width="0.1524" layer="91"/>
+<pinref part="D3" gate="G$1" pin="A"/>
+<wire x1="228.6" y1="165.735" x2="233.68" y2="165.735" width="0.1524" layer="91"/>
 </segment>
 </net>
@@
 <segment>
 <pinref part="R8" gate="G$1" pin="1"/>
-<pinref part="YLW" gate="G$1" pin="A"/>
+<pinref part="D2" gate="G$1" pin="A"/>
 <wire x1="228.6" y1="175.26" x2="233.68" y2="175.26" width="0.1524" layer="91"/>
 </segment>
